File: board/Processor.sch (KiCad schematic (older format))
At the start: 23 parts, among them J3 Conn_01x04, J4 Conn_01x04, J7 Conn_01x02, U1 AMS1117-3V3, U2 STM32F103VETx, Y1 8 MHz, Y2 32.768 kHz

Commit message: Moved around components and added cutouts
Parts:
- U1: LCSC (none) -> C6186
Changed lines of the file:
@@
 $Descr A4 11693 8268
 encoding utf-8
-Sheet 2 9
+Sheet 2 10
 Title ""
 Date ""
@@
 F 5 "Texas Instruments" H 2300 5150 61  0001 C CNN "MFG_NAME"
 F 6 "LM1117" H 2400 5250 61  0001 C CNN "MPN"
+F 7 "C6186" H 2100 5300 60  0001 C CNN "LCSC"
 	1    2100 5300
 	1    0    0    -1
@@
 $EndComp
 $Comp
-L GND #PWR28
+L GND #PWR31
 U 1 1 5EA47061
 P 1900 7000
-F 0 "#PWR28" H 1900 6750 50  0001 C CNN
+F 0 "#PWR31" H 1900 6750 50  0001 C CNN
 F 1 "GND" H 1900 6850 50  0000 C CNN
 F 2 "" H 1900 7000 50  0001 C CNN
@@
 $EndComp
 $Comp
-L GND #PWR30
+L GND #PWR33
 U 1 1 5EA47215
 P 2150 7000
-F 0 "#PWR30" H 2150 6750 50  0001 C CNN
+F 0 "#PWR33" H 2150 6750 50  0001 C CNN
 F 1 "GND" H 2150 6850 50  0000 C CNN
 F 2 "" H 2150 7000 50  0001 C CNN
@@
 $EndComp
 $Comp
-L GND #PWR31
+L GND #PWR34
 U 1 1 5EA4732E
 P 2400 7000
-F 0 "#PWR31" H 2400 6750 50  0001 C CNN
+F 0 "#PWR34" H 2400 6750 50  0001 C CNN
 F 1 "GND" H 2400 6850 50  0000 C CNN
 F 2 "" H 2400 7000 50  0001 C CNN
@@
 $EndComp
 $Comp
-L GND #PWR33
+L GND #PWR36
 U 1 1 5EA4753F
 P 3100 7050
-F 0 "#PWR33" H 3100 6800 50  0001 C CNN
+F 0 "#PWR36" H 3100 6800 50  0001 C CNN
 F 1 "GND" H 3100 6900 50  0000 C CNN
 F 2 "" H 3100 7050 50  0001 C CNN
@@
 $EndComp
 $Comp
-L GND #PWR22
+L GND #PWR25
 U 1 1 5EA47863
 P 1700 5900
-F 0 "#PWR22" H 1700 5650 50  0001 C CNN
+F 0 "#PWR25" H 1700 5650 50  0001 C CNN
 F 1 "GND" H 1700 5750 50  0000 C CNN
 F 2 "" H 1700 5900 50  0001 C CNN
@@
 $EndComp
 $Comp
-L GND #PWR29
+L GND #PWR32
 U 1 1 5EA47964
 P 2100 5900
-F 0 "#PWR29" H 2100 5650 50  0001 C CNN
+F 0 "#PWR32" H 2100 5650 50  0001 C CNN
 F 1 "GND" H 2100 5750 50  0000 C CNN
 F 2 "" H 2100 5900 50  0001 C CNN
@@
 $EndComp
 $Comp
-L +3V3 #PWR32
+L +3V3 #PWR35
 U 1 1 5EA47DD8
 P 2600 5000
-F 0 "#PWR32" H 2600 4850 50  0001 C CNN
+F 0 "#PWR35" H 2600 4850 50  0001 C CNN
 F 1 "+3V3" H 2600 5140 50  0000 C CNN
 F 2 "" H 2600 5000 50  0001 C CNN
@@
 $EndComp
 $Comp
-L +3V3 #PWR27
+L +3V3 #PWR30
 U 1 1 5EA48038
 P 1900 6200
-F 0 "#PWR27" H 1900 6050 50  0001 C CNN
+F 0 "#PWR30" H 1900 6050 50  0001 C CNN
 F 1 "+3V3" H 1900 6340 50  0000 C CNN
 F 2 "" H 1900 6200 50  0001 C CNN
@@
 $EndComp
 $Comp
-L GND #PWR35
+L GND #PWR38
 U 1 1 5EA48BF0
 P 3900 4350
-F 0 "#PWR35" H 3900 4100 50  0001 C CNN
+F 0 "#PWR38" H 3900 4100 50  0001 C CNN
 F 1 "GND" H 3900 4200 50  0000 C CNN
 F 2 "" H 3900 4350 50  0001 C CNN
@@
 $EndComp
 $Comp
-L GND #PWR26
+L GND #PWR29
 U 1 1 5EA4902A
 P 1900 4300
-F 0 "#PWR26" H 1900 4050 50  0001 C CNN
+F 0 "#PWR29" H 1900 4050 50  0001 C CNN
 F 1 "GND" H 1900 4150 50  0000 C CNN
 F 2 "" H 1900 4300 50  0001 C CNN
@@
 $EndComp
 $Comp
-L GND #PWR25
+L GND #PWR28
 U 1 1 5EA49141
 P 1900 3850
-F 0 "#PWR25" H 1900 3600 50  0001 C CNN
+F 0 "#PWR28" H 1900 3600 50  0001 C CNN
 F 1 "GND" H 1900 3700 50  0000 C CNN
 F 2 "" H 1900 3850 50  0001 C CNN
@@
 $EndComp
 $Comp
-L GND #PWR24
+L GND #PWR27
 U 1 1 5EA492E5
 P 1750 3050
-F 0 "#PWR24" H 1750 2800 50  0001 C CNN
+F 0 "#PWR27" H 1750 2800 50  0001 C CNN
 F 1 "GND" H 1750 2900 50  0000 C CNN
 F 2 "" H 1750 3050 50  0001 C CNN
@@
 $EndComp
 $Comp
-L +3V3 #PWR18
+L +3V3 #PWR21
 U 1 1 5EA49507
 P 1200 2700
-F 0 "#PWR18" H 1200 2550 50  0001 C CNN
+F 0 "#PWR21" H 1200 2550 50  0001 C CNN
 F 1 "+3V3" H 1200 2840 50  0000 C CNN
 F 2 "" H 1200 2700 50  0001 C CNN
@@
 $EndComp
 $Comp
-L +3V3 #PWR34
+L +3V3 #PWR37
 U 1 1 5EA4A475
 P 3700 6350
-F 0 "#PWR34" H 3700 6200 50  0001 C CNN
+F 0 "#PWR37" H 3700 6200 50  0001 C CNN
 F 1 "+3V3" H 3700 6490 50  0000 C CNN
 F 2 "" H 3700 6350 50  0001 C CNN
@@
 $EndComp
 $Comp
-L +3V3 #PWR36
+L +3V3 #PWR39
 U 1 1 5EA4A635
 P 3950 6100
-F 0 "#PWR36" H 3950 5950 50  0001 C CNN
+F 0 "#PWR39" H 3950 5950 50  0001 C CNN
 F 1 "+3V3" H 3950 6240 50  0000 C CNN
 F 2 "" H 3950 6100 50  0001 C CNN
@@
 $EndComp
 $Comp
-L +5V #PWR21
+L +5V #PWR24
 U 1 1 5EA47C25
 P 1700 5150
-F 0 "#PWR21" H 1700 5000 50  0001 C CNN
+F 0 "#PWR24" H 1700 5000 50  0001 C CNN
 F 1 "+5V" H 1700 5290 50  0000 C CNN
 F 2 "" H 1700 5150 50  0001 C CNN
@@
 PA10
 $Comp
-L GND #PWR23
+L GND #PWR26
 U 1 1 5EA4912D
 P 1750 2100
-F 0 "#PWR23" H 1750 1850 50  0001 C CNN
+F 0 "#PWR26" H 1750 1850 50  0001 C CNN
 F 1 "GND" H 1750 1950 50  0000 C CNN
 F 2 "" H 1750 2100 50  0001 C CNN
@@
 $EndComp
 $Comp
-L +3V3 #PWR17
+L +3V3 #PWR20
 U 1 1 5EA49133
 P 1200 1750
-F 0 "#PWR17" H 1200 1600 50  0001 C CNN
+F 0 "#PWR20" H 1200 1600 50  0001 C CNN
 F 1 "+3V3" H 1200 1890 50  0000 C CNN
 F 2 "" H 1200 1750 50  0001 C CNN
@@
 Connection ~ 7200 6400
 $Comp
-L GND #PWR41
+L GND #PWR44
 U 1 1 5EA4F93A
 P 6800 6600
-F 0 "#PWR41" H 6800 6350 50  0001 C CNN
+F 0 "#PWR44" H 6800 6350 50  0001 C CNN
 F 1 "GND" H 6800 6450 50  0000 C CNN
 F 2 "" H 6800 6600 50  0001 C CNN
@@
 Connection ~ 7000 6400
 $Comp
-L +3V3 #PWR42
+L +3V3 #PWR45
 U 1 1 5EA4FA98
 P 7800 750
-F 0 "#PWR42" H 7800 600 50  0001 C CNN
+F 0 "#PWR45" H 7800 600 50  0001 C CNN
 F 1 "+3V3" H 7800 890 50  0000 C CNN
 F 2 "" H 7800 750 50  0001 C CNN
@@
 	5150 1400 6100 1400
 $Comp
-L +3V3 #PWR39
+L +3V3 #PWR42
 U 1 1 5EA547A0
 P 5550 1600
-F 0 "#PWR39" H 5550 1450 50  0001 C CNN
+F 0 "#PWR42" H 5550 1450 50  0001 C CNN
 F 1 "+3V3" H 5550 1740 50  0000 C CNN
 F 2 "" H 5550 1600 50  0001 C CNN
@@
 $EndComp
 $Comp
-L GND #PWR40
+L GND #PWR43
 U 1 1 5EA54829
 P 5550 1700
-F 0 "#PWR40" H 5550 1450 50  0001 C CNN
+F 0 "#PWR43" H 5550 1450 50  0001 C CNN
 F 1 "GND" H 5550 1550 50  0000 C CNN
 F 2 "" H 5550 1700 50  0001 C CNN
@@
 $EndComp
 $Comp
-L GND #PWR20
+L GND #PWR23
 U 1 1 5EA5DF96
 P 1600 7000
-F 0 "#PWR20" H 1600 6750 50  0001 C CNN
+F 0 "#PWR23" H 1600 6750 50  0001 C CNN
 F 1 "GND" H 1600 6850 50  0000 C CNN
 F 2 "" H 1600 7000 50  0001 C CNN
@@
 $EndComp
 $Comp
-L GND #PWR19
+L GND #PWR22
 U 1 1 5EA5DFE0
 P 1350 7000
-F 0 "#PWR19" H 1350 6750 50  0001 C CNN
+F 0 "#PWR22" H 1350 6750 50  0001 C CNN
 F 1 "GND" H 1350 6850 50  0000 C CNN
 F 2 "" H 1350 7000 50  0001 C CNN
@@
 $EndComp
 $Comp
-L GND #PWR38
+L GND #PWR41
 U 1 1 5EA71800
 P 5150 1900
-F 0 "#PWR38" H 5150 1650 50  0001 C CNN
+F 0 "#PWR41" H 5150 1650 50  0001 C CNN
 F 1 "GND" H 5150 1750 50  0000 C CNN
 F 2 "" H 5150 1900 50  0001 C CNN
@@
 Connection ~ 5150 1400
 $Comp
-L +3V3 #PWR37
+L +3V3 #PWR40
 U 1 1 5EA72058
 P 5150 650
-F 0 "#PWR37" H 5150 500 50  0001 C CNN
+F 0 "#PWR40" H 5150 500 50  0001 C CNN
 F 1 "+3V3" H 5150 790 50  0000 C CNN
 F 2 "" H 5150 650 50  0001 C CNN
@@
 	5150 650  5150 700
 $Comp
-L GND #PWR43
+L GND #PWR46
 U 1 1 5EA726AB
 P 8900 3150
-F 0 "#PWR43" H 8900 2900 50  0001 C CNN
+F 0 "#PWR46" H 8900 2900 50  0001 C CNN
 F 1 "GND" H 8900 3000 50  0000 C CNN
 F 2 "" H 8900 3150 50  0001 C CNN
